File: zx-bus_board.kicad_pcb (KiCad board)
At the start: 2 copper layers, 101.6 x 98.4 mm, 1328 parts

Commit message: >> Исправил номер ревизии в герберах.
Other:
- board text added: "30.06.22"
- board text added: "REV 0.2"
- board text removed: "27.05.22"
- board text removed: "REV 0.1"
Changed lines of the file:
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@@
     (effects (font (size 1.5 1.5) (thickness 0.3)))
   )
-  (gr_text "27.05.22" (at 250.19 101.6) (layer "B.Cu")
+  (gr_text "30.06.22" (at 250.19 101.6) (layer "B.Cu")
     (effects (font (size 1.5 1.5) (thickness 0.3)) (justify mirror))
   )
-  (gr_text "REV 0.1" (at 160.655 101.6) (layer "B.Cu")
+  (gr_text "REV 0.2" (at 160.655 101.6) (layer "B.Cu")
     (effects (font (size 1.5 1.5) (thickness 0.3)) (justify mirror))
   )
